Commit message: Cleaning up dead code

File: src/scara_description/urdf/scara.urdf.xacro (robot description, xacro)
@@ -42,4 +42,10 @@
             </geometry>
         </visual>
+        <collision>
+            <origin xyz="-0.08 -0.48 1.3" rpy="0 0 0"/>
+            <geometry>
+                <cylinder radius="0.04" length="2.50"/>
+            </geometry>
+        </collision>
         <!-- Rod 3 -->
         <visual>
@@ -49,4 +55,10 @@
             </geometry>
         </visual>
+        <collision>
+            <origin xyz="-0.08 -0.48 1.3" rpy="0 0 0"/>
+            <geometry>
+                <cylinder radius="0.04" length="2.50"/>
+            </geometry>
+        </collision>
         <!-- Threaded Rod -->
         <visual>
@@ -79,4 +91,10 @@
             </geometry>
         </visual>
+        <collision>
+            <origin xyz="0.17 0 1.55" rpy="-${PI/2} 0 -${PI/2}"/>
+            <geometry>
+                <mesh filename="package://scara_description/meshes/Z_BASE.stl" scale="0.01 0.01 0.01"/>
+            </geometry>
+        </collision>
         <xacro:default_inertial mass="1.5"/>
     </link>
@@ -89,4 +107,10 @@
             </geometry>
         </visual>
+        <collision>
+            <origin xyz="-0.015 0.5 -0.4" rpy="${PI/2} 0 0"/>
+            <geometry>
+                <mesh filename="package://scara_description/meshes/ARM_TOP.stl" scale="0.01 0.01 0.01"/>
+            </geometry>
+        </collision>
         <!-- arm bottom -->
         <visual>
@@ -106,5 +130,4 @@
     </link>
     <link name="elbow">
-        <!-- elbow -->
         <!-- elbow hub -->
         <visual>
@@ -121,4 +144,10 @@
             </geometry>
         </visual>
+        <collision>
+            <origin xyz="-0.187 0.245 -0.11" rpy="${PI} 0 ${PI}"/>
+            <geometry>
+                <mesh filename="package://scara_description/meshes/FOREARM.stl" scale="0.01 0.01 0.01"/>
+            </geometry>
+        </collision>
         <xacro:default_inertial mass="1.5"/>
     </link>
@@ -139,14 +168,14 @@
         <parent link="z_base"/>
         <child link="shoulder"/>
-        <origin xyz="0.67 0 -0.07" rpy="0 0 -1.745"/>
+        <origin xyz="0.67 0 -0.07" rpy="0 0 0"/>
         <axis xyz="0 0 1"/>
-        <limit effort="${effort}" velocity="${velocity}" lower="0.0" upper="3.490"/>
+        <limit effort="${effort}" velocity="${velocity}" lower="-1.66" upper="1.66"/>
     </joint>
-        <joint name="joint_3" type="revolute">
+    <joint name="joint_3" type="revolute">
         <parent link="shoulder"/>
         <child link="elbow"/>
-        <origin xyz="0.92 0 0" rpy="0 0 2.269"/>
+        <origin xyz="0.92 0 0" rpy="0 0 0"/>
         <axis xyz="0 0 1"/>
-        <limit effort="${effort}" velocity="${velocity}" lower="-4.538" upper="0.0"/>
+        <limit effort="${effort}" velocity="${velocity}" lower="-2.37" upper="2.37"/>
     </joint>
 </robot>

File: src/scara_description/urdf/scara_gazebo.xacro (robot description, xacro)
@@ -1,38 +1,8 @@
 <?xml version="1.0"?>
-<robot xmlns:xacro="http://www.ros.org/wiki/xacro" name="scara">
+<robot xmlns:xacro="http://www.ros.org/wiki/xacro" name="SCARA">
     <gazebo>
-        <!--
-        <plugin filename="gz-sim-sensors-system" name="gz::sim::systems::Sensors">
-            <render_engine>ogre2</render_engine>
-        </plugin>
-        -->
         <plugin filename="gz_ros2_control-system" name="gz_ros2_control::GazeboSimROS2ControlPlugin">
             <parameters>$(find scara_controller)/config/scara_controllers.yaml</parameters>
         </plugin>
     </gazebo>
-    <!--
-    <link name="camera_link_optical"></link>
-    <gazebo reference="rgb_camera">
-        <sensor name="camera" type="camera">
-            <pose> 0 0 0 0 0 0 </pose>
-            <visualize>true</visualize>
-            <update_rate>10</update_rate>
-            <camera>
-                <camera_info_topic>camera/camera_info</camera_info_topic>
-                <horizontal_fov>1.21126</horizontal_fov>
-                <image>
-                    <format>R8G8B8</format>
-                    <width>2304</width>
-                    <height>1296</height>
-                </image>
-                <clip>
-                    <near>0.05</near>
-                    <far>5.0</far>
-                </clip>
-            </camera>
-            <topic>camera/image_raw</topic>
-            <gz_frame_id>camera_link_optical</gz_frame_id>
-        </sensor>
-    </gazebo>
--->
 </robot>

File: src/scara_description/urdf/scara_ros2_control.xacro (robot description, xacro)
@@ -1,4 +1,4 @@
 <?xml version="1.0"?>
-<robot xmlns:xacro="http://www.ros.org/wiki/xacro" name="scara">
+<robot xmlns:xacro="http://www.ros.org/wiki/xacro" name="SCARA">
     <xacro:property name="PI" value="3.14159265359" />
     <ros2_control type="system" name="RobotSystem">
@@ -15,6 +15,6 @@
         <joint name="joint_2">
             <command_interface name="position">
-                <param name="min">0.0</param>
-                <param name="max">3.490</param>
+                <param name="min">-1.66</param>
+                <param name="max">1.66</param>
             </command_interface>
             <state_interface name="position"/>
@@ -22,9 +22,20 @@
         <joint name="joint_3">
             <command_interface name="position">
-                <param name="min">-4.538</param>
-                <param name="max">0.0</param>
+                <param name="min">-2.37</param>
+                <param name="max">2.37</param>
             </command_interface>
             <state_interface name="position"/>
         </joint>
     </ros2_control>
+    <!-- Transmissions -->
+    <transmission name="trans_joint_1">
+        <type>transmission_interface/SimpleTransmission</type>
+        <joint name="joint_1">
+          <hardwareInterface>hardware_interface/PositionJointInterface</hardwareInterface>
+        </joint>
+        <actuator name="motor_joint_1">
+          <hardwareInterface>hardware_interface/PositionJointInterface</hardwareInterface>
+          <mechanicalReduction>1.0</mechanicalReduction>
+        </actuator>
+    </transmission>
 </robot>

Commit message: changes due to out-of-bounds joint-1

File: src/scara_description/urdf/scara.urdf.xacro (robot description, xacro)
@@ -163,5 +163,7 @@
         <origin xyz="0 0 0.9" rpy="0 0 0"/>
         <axis xyz="0 0 1"/>
-        <limit effort="${effort}" velocity="${velocity}" lower="0.0" upper="1.47"/>
+        <!--<limit effort="${effort}" velocity="${velocity}" lower="0.0" upper="1.47"/>-->
+        <limit effort="1000" velocity="10" lower="0.0" upper="1.47"/>
+        <dynamics damping="0.5" friction="0.5"/>
     </joint>
     <joint name="joint_2" type="revolute">

Commit message: added gripper prototype

File: src/scara_description/urdf/scara.urdf.xacro (robot description, xacro)
@@ -152,4 +152,40 @@
         <xacro:default_inertial mass="1.5"/>
     </link>
+    <link name="gripper_base">
+        <visual>
+            <origin xyz="0 0 -0.15" rpy="${PI} 0 ${PI}"/>
+            <geometry>
+                <cylinder radius="0.12" length="0.1"/>
+            </geometry>
+        </visual>
+        <collision>
+            <origin xyz="0 0 0" rpy="${PI} 0 ${PI}"/>
+            <geometry>
+                <cylinder radius="0.04" length="0.5"/>
+            </geometry>
+        </collision>
+        <xacro:default_inertial mass="1.5"/>
+    </link>
+    <link name="gripper">
+        <visual>
+            <origin xyz="0 0 -0.3" rpy="${PI} 0 ${PI}"/>
+            <geometry>
+                <cylinder radius="0.04" length="0.5"/>
+            </geometry>
+        </visual>
+        <visual>
+            <origin xyz="0.1 0 -0.5" rpy="${PI} 0 ${PI}"/>
+            <geometry>
+                <box size="0.2 0.01 0.1"/>
+            </geometry>
+        </visual>
+        <collision>
+            <origin xyz="0 0 0" rpy="${PI} 0 ${PI}"/>
+            <geometry>
+                <cylinder radius="0.04" length="0.5"/>
+            </geometry>
+        </collision>
+        <xacro:default_inertial mass="1.5"/>
+    </link>
     <!-- joints -->
     <joint name="virtual_joint" type="fixed">
@@ -181,3 +217,15 @@
         <limit effort="${effort}" velocity="${velocity}" lower="-2.37" upper="2.37"/>
     </joint>
+    <joint name="joint_4" type="revolute">
+        <parent link="elbow"/>
+        <child link="gripper_base"/>
+        <origin xyz="1.2 0 0" rpy="0 0 0"/>
+        <axis xyz="0 0 1"/>
+        <limit effort="${effort}" velocity="${velocity}" lower="-${PI}" upper="${PI}"/>
+    </joint>
+    <joint name="joint_5" type="fixed">
+        <parent link="gripper_base"/>
+        <child link="gripper"/>
+        <origin xyz="0 0 -0.1" rpy="0 0 0"/>
+    </joint>
 </robot>

File: src/scara_description/urdf/scara_ros2_control.xacro (robot description, xacro)
@@ -27,4 +27,11 @@
             <state_interface name="position"/>
         </joint>
+        <joint name="joint_4">
+            <command_interface name="position">
+                <param name="min">-${PI}</param>
+                <param name="max">${PI}</param>
+            </command_interface>
+            <state_interface name="position"/>
+        </joint>
     </ros2_control>
     <!-- Transmissions -->

Commit message: adjusting urdf to real robot size, adjusting hardcoded positions

File: src/scara_description/urdf/scara.urdf.xacro (robot description, xacro)
@@ -23,61 +23,61 @@
         <!-- Base Mesh -->
         <visual>
-            <origin xyz="0.17 0 0" rpy="${PI/2} 0 ${PI/2}"/>
-            <geometry>
-                <mesh filename="package://scara_description/meshes/BASEPLATE.stl" scale="0.01 0.01 0.01"/>
+            <origin xyz="0.017 0 0" rpy="${PI/2} 0 ${PI/2}"/>
+            <geometry>
+                <mesh filename="package://scara_description/meshes/BASEPLATE.stl" scale="0.001 0.001 0.001"/>
             </geometry>
         </visual>
         <!-- Rod 1 -->
         <visual>
-            <origin xyz="0.67 0 1.3" rpy="0 0 0"/>
-            <geometry>
-                <cylinder radius="0.04" length="2.50"/>
+            <origin xyz="0.067 0 0.13" rpy="0 0 0"/>
+            <geometry>
+                <cylinder radius="0.004" length="0.250"/>
             </geometry>
         </visual>
         <!-- Rod 2 -->
         <visual>
-            <origin xyz="-0.08 0.48 1.3" rpy="0 0 0"/>
-            <geometry>
-                <cylinder radius="0.04" length="2.50"/>
-            </geometry>
-        </visual>
-        <collision>
-            <origin xyz="-0.08 -0.48 1.3" rpy="0 0 0"/>
-            <geometry>
-                <cylinder radius="0.04" length="2.50"/>
+            <origin xyz="-0.008 0.048 0.13" rpy="0 0 0"/>
+            <geometry>
+                <cylinder radius="0.004" length="0.250"/>
+            </geometry>
+        </visual>
+        <collision>
+            <origin xyz="-0.008 -0.048 0.13" rpy="0 0 0"/>
+            <geometry>
+                <cylinder radius="0.004" length="0.250"/>
             </geometry>
         </collision>
         <!-- Rod 3 -->
         <visual>
-            <origin xyz="-0.08 -0.48 1.3" rpy="0 0 0"/>
-            <geometry>
-                <cylinder radius="0.04" length="2.50"/>
-            </geometry>
-        </visual>
-        <collision>
-            <origin xyz="-0.08 -0.48 1.3" rpy="0 0 0"/>
-            <geometry>
-                <cylinder radius="0.04" length="2.50"/>
+            <origin xyz="-0.008 -0.048 0.13" rpy="0 0 0"/>
+            <geometry>
+                <cylinder radius="0.004" length="0.250"/>
+            </geometry>
+        </visual>
+        <collision>
+            <origin xyz="-0.008 -0.048 0.13" rpy="0 0 0"/>
+            <geometry>
+                <cylinder radius="0.004" length="0.250"/>
             </geometry>
         </collision>
         <!-- Threaded Rod -->
         <visual>
-            <origin xyz="0 0 1.3" rpy="0 0 0"/>
-            <geometry>
-                <cylinder radius="0.04" length="2.50"/>
+            <origin xyz="0 0 0.13" rpy="0 0 0"/>
+            <geometry>
+                <cylinder radius="0.004" length="0.250"/>
             </geometry>
         </visual>
         <!-- Base cover -->
         <visual>
-            <origin xyz="0.17 0 3.08" rpy="-${PI/2} 0 -${PI/2}"/>
-            <geometry>
-                <mesh filename="package://scara_description/meshes/TOP_TRIANGLE.stl" scale="0.01 0.01 0.01"/>
+            <origin xyz="0.017 0 0.308" rpy="-${PI/2} 0 -${PI/2}"/>
+            <geometry>
+                <mesh filename="package://scara_description/meshes/TOP_TRIANGLE.stl" scale="0.001 0.001 0.001"/>
             </geometry>
         </visual>
         <!-- Motors triangle -->
         <visual>
-            <origin xyz="0.17 0 3.1" rpy="-${PI/2} 0 -${PI/2}"/>
-            <geometry>
-                <mesh filename="package://scara_description/meshes/MOTORS_TRIANGLE.stl" scale="0.01 0.01 0.01"/>
+            <origin xyz="0.017 0 0.31" rpy="-${PI/2} 0 -${PI/2}"/>
+            <geometry>
+                <mesh filename="package://scara_description/meshes/MOTORS_TRIANGLE.stl" scale="0.001 0.001 0.001"/>
             </geometry>
         </visual>
@@ -86,13 +86,13 @@
     <link name="z_base">
         <visual>
-            <origin xyz="0.17 0 1.55" rpy="-${PI/2} 0 -${PI/2}"/>
-            <geometry>
-                <mesh filename="package://scara_description/meshes/Z_BASE.stl" scale="0.01 0.01 0.01"/>
-            </geometry>
-        </visual>
-        <collision>
-            <origin xyz="0.17 0 1.55" rpy="-${PI/2} 0 -${PI/2}"/>
-            <geometry>
-                <mesh filename="package://scara_description/meshes/Z_BASE.stl" scale="0.01 0.01 0.01"/>
+            <origin xyz="0.017 0 0.155" rpy="-${PI/2} 0 -${PI/2}"/>
+            <geometry>
+                <mesh filename="package://scara_description/meshes/Z_BASE.stl" scale="0.001 0.001 0.001"/>
+            </geometry>
+        </visual>
+        <collision>
+            <origin xyz="0.017 0 0.155" rpy="-${PI/2} 0 -${PI/2}"/>
+            <geometry>
+                <mesh filename="package://scara_description/meshes/Z_BASE.stl" scale="0.001 0.001 0.001"/>
             </geometry>
         </collision>
@@ -102,27 +102,27 @@
         <!-- arm top -->
         <visual>
-            <origin xyz="-0.015 0.5 -0.4" rpy="${PI/2} 0 0"/>
-            <geometry>
-                <mesh filename="package://scara_description/meshes/ARM_TOP.stl" scale="0.01 0.01 0.01"/>
-            </geometry>
-        </visual>
-        <collision>
-            <origin xyz="-0.015 0.5 -0.4" rpy="${PI/2} 0 0"/>
-            <geometry>
-                <mesh filename="package://scara_description/meshes/ARM_TOP.stl" scale="0.01 0.01 0.01"/>
+            <origin xyz="-0.0015 0.05 -0.04" rpy="${PI/2} 0 0"/>
+            <geometry>
+                <mesh filename="package://scara_description/meshes/ARM_TOP.stl" scale="0.001 0.001 0.001"/>
+            </geometry>
+        </visual>
+        <collision>
+            <origin xyz="-0.0015 0.05 -0.04" rpy="${PI/2} 0 0"/>
+            <geometry>
+                <mesh filename="package://scara_description/meshes/ARM_TOP.stl" scale="0.001 0.001 0.001"/>
             </geometry>
         </collision>
         <!-- arm bottom -->
         <visual>
-            <origin xyz="0.49 0 -0.44" rpy="${PI/2} 0 -${PI/2} "/>
-            <geometry>
-                <mesh filename="package://scara_description/meshes/ARM_BOTTOM.stl" scale="0.01 0.01 0.01"/>
+            <origin xyz="0.049 0 -0.044" rpy="${PI/2} 0 -${PI/2} "/>
+            <geometry>
+                <mesh filename="package://scara_description/meshes/ARM_BOTTOM.stl" scale="0.001 0.001 0.001"/>
             </geometry>
         </visual>
         <!-- reduction -->
         <visual>
-            <origin xyz="0.18 -0.245 -0.07" rpy="${PI} 0 0"/>
-            <geometry>
-                <mesh filename="package://scara_description/meshes/REDUCTION.stl" scale="0.01 0.01 0.01"/>
+            <origin xyz="0.018 -0.0245 -0.007" rpy="${PI} 0 0"/>
+            <geometry>
+                <mesh filename="package://scara_description/meshes/REDUCTION.stl" scale="0.001 0.001 0.001"/>
             </geometry>
         </visual>
@@ -132,20 +132,20 @@
         <!-- elbow hub -->
         <visual>
-            <origin xyz="-0.187 0.245 -0.11" rpy="${PI} 0 ${PI}"/>
-            <geometry>
-                <mesh filename="package://scara_description/meshes/ARM_HUB.stl" scale="0.01 0.01 0.01"/>
+            <origin xyz="-0.0187 0.0245 -0.011" rpy="${PI} 0 ${PI}"/>
+            <geometry>
+                <mesh filename="package://scara_description/meshes/ARM_HUB.stl" scale="0.001 0.001 0.001"/>
             </geometry>
         </visual>
         <!-- elbow arm -->
         <visual>
-            <origin xyz="-0.187 0.245 -0.11" rpy="${PI} 0 ${PI}"/>
-            <geometry>
-                <mesh filename="package://scara_description/meshes/FOREARM.stl" scale="0.01 0.01 0.01"/>
-            </geometry>
-        </visual>
-        <collision>
-            <origin xyz="-0.187 0.245 -0.11" rpy="${PI} 0 ${PI}"/>
-            <geometry>
-                <mesh filename="package://scara_description/meshes/FOREARM.stl" scale="0.01 0.01 0.01"/>
+            <origin xyz="-0.0187 0.0245 -0.011" rpy="${PI} 0 ${PI}"/>
+            <geometry>
+                <mesh filename="package://scara_description/meshes/FOREARM.stl" scale="0.001 0.001 0.001"/>
+            </geometry>
+        </visual>
+        <collision>
+            <origin xyz="-0.0187 0.0245 -0.011" rpy="${PI} 0 ${PI}"/>
+            <geometry>
+                <mesh filename="package://scara_description/meshes/FOREARM.stl" scale="0.001 0.001 0.001"/>
             </geometry>
         </collision>
@@ -154,7 +154,28 @@
     <link name="gripper_base">
         <visual>
-            <origin xyz="0 0 -0.15" rpy="${PI} 0 ${PI}"/>
-            <geometry>
-                <cylinder radius="0.12" length="0.1"/>
+            <origin xyz="0 0 -0.015" rpy="${PI} 0 ${PI}"/>
+            <geometry>
+                <cylinder radius="0.012" length="0.01"/>
+            </geometry>
+        </visual>
+        <collision>
+            <origin xyz="0 0 -0.015" rpy="${PI} 0 ${PI}"/>
+            <geometry>
+                <cylinder radius="0.004" length="0.05"/>
+            </geometry>
+        </collision>
+        <xacro:default_inertial mass="1.5"/>
+    </link>
+    <link name="gripper">
+        <visual>
+            <origin xyz="0 0 -0.03" rpy="${PI} 0 ${PI}"/>
+            <geometry>
+                <cylinder radius="0.004" length="0.05"/>
+            </geometry>
+        </visual>
+        <visual>
+            <origin xyz="0.01 0 -0.05" rpy="${PI} 0 ${PI}"/>
+            <geometry>
+                <box size="0.02 0.001 0.01"/>
             </geometry>
         </visual>
@@ -162,26 +183,5 @@
             <origin xyz="0 0 0" rpy="${PI} 0 ${PI}"/>
             <geometry>
-                <cylinder radius="0.04" length="0.5"/>
-            </geometry>
-        </collision>
-        <xacro:default_inertial mass="1.5"/>
-    </link>
-    <link name="gripper">
-        <visual>
-            <origin xyz="0 0 -0.3" rpy="${PI} 0 ${PI}"/>
-            <geometry>
-                <cylinder radius="0.04" length="0.5"/>
-            </geometry>
-        </visual>
-        <visual>
-            <origin xyz="0.1 0 -0.5" rpy="${PI} 0 ${PI}"/>
-            <geometry>
-                <box size="0.2 0.01 0.1"/>
-            </geometry>
-        </visual>
-        <collision>
-            <origin xyz="0 0 0" rpy="${PI} 0 ${PI}"/>
-            <geometry>
-                <cylinder radius="0.04" length="0.5"/>
+                <cylinder radius="0.004" length="0.05"/>
             </geometry>
         </collision>
@@ -197,8 +197,8 @@
         <parent link="base_link"/>
         <child link="z_base"/>
-        <origin xyz="0 0 0.9" rpy="0 0 0"/>
+        <origin xyz="0 0 0.09" rpy="0 0 0"/>
         <axis xyz="0 0 1"/>
         <!--<limit effort="${effort}" velocity="${velocity}" lower="0.0" upper="1.47"/>-->
-        <limit effort="1000" velocity="10" lower="0.0" upper="1.47"/>
+        <limit effort="1000" velocity="10" lower="0.0" upper="0.147"/>
         <dynamics damping="0.5" friction="0.5"/>
     </joint>
@@ -206,5 +206,5 @@
         <parent link="z_base"/>
         <child link="shoulder"/>
-        <origin xyz="0.67 0 -0.07" rpy="0 0 0"/>
+        <origin xyz="0.067 0 -0.007" rpy="0 0 0"/>
         <axis xyz="0 0 1"/>
         <limit effort="${effort}" velocity="${velocity}" lower="-1.66" upper="1.66"/>
@@ -213,5 +213,5 @@
         <parent link="shoulder"/>
         <child link="elbow"/>
-        <origin xyz="0.92 0 0" rpy="0 0 0"/>
+        <origin xyz="0.092 0 0" rpy="0 0 0"/>
         <axis xyz="0 0 1"/>
         <limit effort="${effort}" velocity="${velocity}" lower="-2.37" upper="2.37"/>
@@ -220,5 +220,5 @@
         <parent link="elbow"/>
         <child link="gripper_base"/>
-        <origin xyz="1.2 0 0" rpy="0 0 0"/>
+        <origin xyz="0.12 0 0" rpy="0 0 0"/>
         <axis xyz="0 0 1"/>
         <limit effort="${effort}" velocity="${velocity}" lower="-${PI}" upper="${PI}"/>
@@ -227,5 +227,5 @@
         <parent link="gripper_base"/>
         <child link="gripper"/>
-        <origin xyz="0 0 -0.1" rpy="0 0 0"/>
+        <origin xyz="0 0 -0.01" rpy="0 0 0"/>
     </joint>
 </robot>

Commit message: Adjusting joint_3 lower and upper limit according to documentation

File: src/scara_description/urdf/scara.urdf.xacro (robot description, xacro)
@@ -216,5 +216,5 @@
         <origin xyz="0.092 0 0" rpy="0 0 0"/>
         <axis xyz="0 0 1"/>
-        <limit effort="${effort}" velocity="${velocity}" lower="-2.37" upper="2.37"/>
+        <limit effort="${effort}" velocity="${velocity}" lower="-2.44" upper="2.44"/>
     </joint>
     <joint name="joint_4" type="revolute">
