Commit message: changes in physical robot model after first real build

File: src/scara_description/urdf/scara.urdf.xacro (robot description, xacro)
@@ -103,25 +103,25 @@
         <!-- arm top -->
         <visual>
-            <origin xyz="-0.0015 0.05 -0.04" rpy="${PI/2} 0 0"/>
-            <geometry>
-                <mesh filename="package://scara_description/meshes/ARM_TOP.stl" scale="0.001 0.001 0.001"/>
-            </geometry>
-        </visual>
-        <collision>
-            <origin xyz="-0.0015 0.05 -0.04" rpy="${PI/2} 0 0"/>
-            <geometry>
-                <mesh filename="package://scara_description/meshes/ARM_TOP.stl" scale="0.001 0.001 0.001"/>
+            <origin xyz="0 0 0" rpy="0 0 0"/>
+            <geometry>
+                <mesh filename="package://scara_description/meshes/MY_ARM_TOP.stl" scale="0.001 0.001 0.001"/>
+            </geometry>
+        </visual>
+        <collision>
+            <origin xyz="0 0 0" rpy="0 0 0"/>
+            <geometry>
+                <mesh filename="package://scara_description/meshes/MY_ARM_TOP.stl" scale="0.001 0.001 0.001"/>
             </geometry>
         </collision>
         <!-- arm bottom -->
         <visual>
-            <origin xyz="0.049 0 -0.044" rpy="${PI/2} 0 -${PI/2} "/>
-            <geometry>
-                <mesh filename="package://scara_description/meshes/ARM_BOTTOM.stl" scale="0.001 0.001 0.001"/>
+            <origin xyz="0 0 -0.029" rpy="${PI/2} 0 -${PI/2} "/>
+            <geometry>
+                <mesh filename="package://scara_description/meshes/MY_ARM_BOTTOM.stl" scale="0.001 0.001 0.001"/>
             </geometry>
         </visual>
         <!-- reduction -->
         <visual>
-            <origin xyz="0.018 -0.0245 -0.007" rpy="${PI} 0 0"/>
+            <origin xyz="0.018 -0.0245 -0.0005" rpy="${PI} 0 0"/>
             <geometry>
                 <mesh filename="package://scara_description/meshes/REDUCTION.stl" scale="0.001 0.001 0.001"/>
@@ -133,5 +133,5 @@
         <!-- elbow hub -->
         <visual>
-            <origin xyz="-0.0187 0.0245 -0.011" rpy="${PI} 0 ${PI}"/>
+            <origin xyz="-0.0183 0.0242 0" rpy="${PI} 0 ${PI}"/>
             <geometry>
                 <mesh filename="package://scara_description/meshes/ARM_HUB.stl" scale="0.001 0.001 0.001"/>
@@ -140,13 +140,34 @@
         <!-- elbow arm -->
         <visual>
-            <origin xyz="-0.0187 0.0245 -0.011" rpy="${PI} 0 ${PI}"/>
-            <geometry>
-                <mesh filename="package://scara_description/meshes/FOREARM.stl" scale="0.001 0.001 0.001"/>
-            </geometry>
-        </visual>
-        <collision>
-            <origin xyz="-0.0187 0.0245 -0.011" rpy="${PI} 0 ${PI}"/>
-            <geometry>
-                <mesh filename="package://scara_description/meshes/FOREARM.stl" scale="0.001 0.001 0.001"/>
+            <origin xyz="0 0 -0.003" rpy="${PI/2} 0 -${PI/2}"/>
+            <geometry>
+                <mesh filename="package://scara_description/meshes/MY_FOREARM.stl" scale="0.001 0.001 0.001"/>
+            </geometry>
+        </visual>
+        <!-- camera base-->
+        <visual>
+            <origin xyz="0.1625 0.0195 0.011" rpy="${PI/2} 0 ${PI/2}"/>
+            <geometry>
+                <mesh filename="package://scara_description/meshes/MY_CAMERA_BASE.stl" scale="0.001 0.001 0.001"/>
+            </geometry>
+        </visual>
+        <!-- camera -->
+        <visual>
+            <origin xyz="0.173 0.0195 0.011" rpy="${PI} 0 -${PI/2}"/>
+            <geometry>
+                <mesh filename="package://scara_description/meshes/CAMERA.stl" scale="0.001 0.001 0.001"/>
+            </geometry>
+        </visual>
+        <collision>
+            <origin xyz="0 0 -0.003" rpy="${PI/2} 0 -${PI/2}"/>
+            <geometry>
+                <mesh filename="package://scara_description/meshes/MY_FOREARM.stl" scale="0.001 0.001 0.001"/>
+            </geometry>
+        </collision>
+        <xacro:default_inertial mass="1.5"/>
+        <collision>
+            <origin xyz="0.1625 0.0195 0.011" rpy="${PI/2} 0 ${PI/2}"/>
+            <geometry>
+                <mesh filename="package://scara_description/meshes/MY_CAMERA_BASE.stl" scale="0.001 0.001 0.001"/>
             </geometry>
         </collision>
@@ -155,32 +176,32 @@
     <link name="gripper_base">
         <visual>
+            <origin xyz="0 0 -0.0305" rpy="${PI/2} 0 0"/>
+            <geometry>
+                <mesh filename="package://scara_description/meshes/MY_GRIPPER_GEAR.stl" scale="0.001 0.001 0.001"/>
+            </geometry>
+        </visual>
+        <collision>
+            <origin xyz="0 0 -0.0305" rpy="${PI/2} 0 0"/>
+            <geometry>
+                <cylinder radius="0.004" length="0.05"/>
+            </geometry>
+        </collision>
+        <xacro:default_inertial mass="1.5"/>
+    </link>
+    <link name="gripper">
+        <visual>
             <origin xyz="0 0 -0.015" rpy="${PI} 0 ${PI}"/>
             <geometry>
-                <cylinder radius="0.012" length="0.01"/>
+                <cylinder radius="0.004" length="0.065"/>
+            </geometry>
+        </visual>
+        <visual>
+            <origin xyz="0.005 0 -0.040" rpy="${PI} 0 ${PI}"/>
+            <geometry>
+                <box size="0.01 0.001 0.01"/>
             </geometry>
         </visual>
         <collision>
             <origin xyz="0 0 -0.015" rpy="${PI} 0 ${PI}"/>
-            <geometry>
-                <cylinder radius="0.004" length="0.05"/>
-            </geometry>
-        </collision>
-        <xacro:default_inertial mass="1.5"/>
-    </link>
-    <link name="gripper">
-        <visual>
-            <origin xyz="0 0 -0.03" rpy="${PI} 0 ${PI}"/>
-            <geometry>
-                <cylinder radius="0.004" length="0.05"/>
-            </geometry>
-        </visual>
-        <visual>
-            <origin xyz="0.01 0 -0.05" rpy="${PI} 0 ${PI}"/>
-            <geometry>
-                <box size="0.02 0.001 0.01"/>
-            </geometry>
-        </visual>
-        <collision>
-            <origin xyz="0 0 0" rpy="${PI} 0 ${PI}"/>
             <geometry>
                 <cylinder radius="0.004" length="0.05"/>
@@ -198,8 +219,7 @@
         <parent link="base_link"/>
         <child link="z_base"/>
-        <origin xyz="0 0 0.09" rpy="0 0 0"/>
-        <axis xyz="0 0 1"/>
-        <!--<limit effort="${effort}" velocity="${velocity}" lower="0.0" upper="1.47"/>-->
-        <limit effort="1000" velocity="10" lower="0.0" upper="0.147"/>
+        <origin xyz="0 0 0.239" rpy="0 0 0"/>
+        <axis xyz="0 0 1"/>
+        <limit effort="1000" velocity="10" lower="-0.143" upper="0.0"/>
         <dynamics damping="0.5" friction="0.5"/>
     </joint>
@@ -207,19 +227,19 @@
         <parent link="z_base"/>
         <child link="shoulder"/>
-        <origin xyz="0.067 0 -0.007" rpy="0 0 0"/>
-        <axis xyz="0 0 1"/>
-        <limit effort="${effort}" velocity="${velocity}" lower="-1.66" upper="1.66"/>
+        <origin xyz="0.067 0 -0.0125" rpy="0 0 1.98"/>
+        <axis xyz="0 0 1"/>
+        <limit effort="${effort}" velocity="${velocity}" lower="-3.96" upper="0.0"/>
     </joint>
     <joint name="joint_3" type="revolute">
         <parent link="shoulder"/>
         <child link="elbow"/>
-        <origin xyz="0.092 0 0" rpy="0 0 0"/>
-        <axis xyz="0 0 1"/>
-        <limit effort="${effort}" velocity="${velocity}" lower="-2.44" upper="2.44"/>
+        <origin xyz="0.092 0 -0.006" rpy="0 0 -2.27"/>
+        <axis xyz="0 0 1"/>
+        <limit effort="${effort}" velocity="${velocity}" lower="0.0" upper="4.54"/>
     </joint>
     <joint name="joint_4" type="revolute">
         <parent link="elbow"/>
         <child link="gripper_base"/>
-        <origin xyz="0.12 0 0" rpy="0 0 0"/>
+        <origin xyz="0.1 0 0" rpy="0 0 0"/>
         <axis xyz="0 0 1"/>
         <limit effort="${effort}" velocity="${velocity}" lower="-${PI}" upper="${PI}"/>
@@ -228,5 +248,5 @@
         <parent link="gripper_base"/>
         <child link="gripper"/>
-        <origin xyz="0 0 -0.01" rpy="0 0 0"/>
+        <origin xyz="0 0 0" rpy="0 0 0"/>
     </joint>
 </robot>

Commit message: Working demo with my own written IK node

File: src/scara_description/urdf/scara.urdf.xacro (robot description, xacro)
@@ -184,5 +184,5 @@
             <origin xyz="0 0 -0.0305" rpy="${PI/2} 0 0"/>
             <geometry>
-                <cylinder radius="0.004" length="0.05"/>
+                <mesh filename="package://scara_description/meshes/MY_GRIPPER_GEAR.stl" scale="0.001 0.001 0.001"/>
             </geometry>
         </collision>
@@ -227,14 +227,18 @@
         <parent link="z_base"/>
         <child link="shoulder"/>
-        <origin xyz="0.067 0 -0.0125" rpy="0 0 1.98"/>
-        <axis xyz="0 0 1"/>
-        <limit effort="${effort}" velocity="${velocity}" lower="-3.96" upper="0.0"/>
+        <!--<origin xyz="0.067 0 -0.0125" rpy="0 0 1.98"/>-->
+        <origin xyz="0.067 0 -0.0125" rpy="0 0 0"/>
+        <axis xyz="0 0 1"/>
+        <limit effort="${effort}" velocity="${velocity}" lower="-1.98" upper="1.98"/>
+        <!--<limit effort="${effort}" velocity="${velocity}" lower="-3.96" upper="0.0"/>-->
     </joint>
     <joint name="joint_3" type="revolute">
         <parent link="shoulder"/>
         <child link="elbow"/>
-        <origin xyz="0.092 0 -0.006" rpy="0 0 -2.27"/>
-        <axis xyz="0 0 1"/>
-        <limit effort="${effort}" velocity="${velocity}" lower="0.0" upper="4.54"/>
+        <!--<origin xyz="0.092 0 -0.006" rpy="0 0 -2.27"/>-->
+        <origin xyz="0.092 0 -0.006" rpy="0 0 0"/>
+        <axis xyz="0 0 1"/>
+        <limit effort="${effort}" velocity="${velocity}" lower="-2.27" upper="2.27"/>
+        <!--<limit effort="${effort}" velocity="${velocity}" lower="0.0" upper="4.54"/>-->
     </joint>
     <joint name="joint_4" type="revolute">

File: src/scara_description/urdf/scara_ros2_control.xacro (robot description, xacro)
@@ -30,44 +30,3 @@
     </joint>
   </ros2_control>
-  <!-- Transmissions for all joints -->
-  <transmission name="trans_joint_1">
-    <type>transmission_interface/SimpleTransmission</type>
-    <joint name="joint_1">
-      <hardwareInterface>hardware_interface/PositionJointInterface</hardwareInterface>
-    </joint>
-    <actuator name="motor_joint_1">
-      <hardwareInterface>hardware_interface/PositionJointInterface</hardwareInterface>
-      <mechanicalReduction>1.0</mechanicalReduction>
-    </actuator>
-  </transmission>
-  <transmission name="trans_joint_2">
-    <type>transmission_interface/SimpleTransmission</type>
-    <joint name="joint_2">
-      <hardwareInterface>hardware_interface/PositionJointInterface</hardwareInterface>
-    </joint>
-    <actuator name="motor_joint_2">
-      <hardwareInterface>hardware_interface/PositionJointInterface</hardwareInterface>
-      <mechanicalReduction>1.0</mechanicalReduction>
-    </actuator>
-  </transmission>
-  <transmission name="trans_joint_3">
-    <type>transmission_interface/SimpleTransmission</type>
-    <joint name="joint_3">
-      <hardwareInterface>hardware_interface/PositionJointInterface</hardwareInterface>
-    </joint>
-    <actuator name="motor_joint_3">
-      <hardwareInterface>hardware_interface/PositionJointInterface</hardwareInterface>
-      <mechanicalReduction>1.0</mechanicalReduction>
-    </actuator>
-  </transmission>
-  <transmission name="trans_joint_4">
-    <type>transmission_interface/SimpleTransmission</type>
-    <joint name="joint_4">
-      <hardwareInterface>hardware_interface/PositionJointInterface</hardwareInterface>
-    </joint>
-    <actuator name="motor_joint_4">
-      <hardwareInterface>hardware_interface/PositionJointInterface</hardwareInterface>
-      <mechanicalReduction>1.0</mechanicalReduction>
-    </actuator>
-  </transmission>
 </robot>

Commit message: Finished moving to non-moveit solution. Passed physical tests.

File: src/scara_description/urdf/scara.urdf.xacro (robot description, xacro)
@@ -103,5 +103,5 @@
         <!-- arm top -->
         <visual>
-            <origin xyz="0 0 0" rpy="0 0 0"/>
+            <origin xyz="0 0 -0.0125" rpy="0 0 0"/>
             <geometry>
                 <mesh filename="package://scara_description/meshes/MY_ARM_TOP.stl" scale="0.001 0.001 0.001"/>
@@ -109,5 +109,5 @@
         </visual>
         <collision>
-            <origin xyz="0 0 0" rpy="0 0 0"/>
+            <origin xyz="0 0 -0.0125" rpy="0 0 0"/>
             <geometry>
                 <mesh filename="package://scara_description/meshes/MY_ARM_TOP.stl" scale="0.001 0.001 0.001"/>
@@ -116,5 +116,5 @@
         <!-- arm bottom -->
         <visual>
-            <origin xyz="0 0 -0.029" rpy="${PI/2} 0 -${PI/2} "/>
+            <origin xyz="0 0 -0.0415" rpy="${PI/2} 0 -${PI/2} "/>
             <geometry>
                 <mesh filename="package://scara_description/meshes/MY_ARM_BOTTOM.stl" scale="0.001 0.001 0.001"/>
@@ -123,5 +123,5 @@
         <!-- reduction -->
         <visual>
-            <origin xyz="0.018 -0.0245 -0.0005" rpy="${PI} 0 0"/>
+            <origin xyz="0.018 -0.0245 -0.0130" rpy="${PI} 0 0"/>
             <geometry>
                 <mesh filename="package://scara_description/meshes/REDUCTION.stl" scale="0.001 0.001 0.001"/>
@@ -133,5 +133,5 @@
         <!-- elbow hub -->
         <visual>
-            <origin xyz="-0.0183 0.0242 0" rpy="${PI} 0 ${PI}"/>
+            <origin xyz="-0.0183 0.0242 -0.0185" rpy="${PI} 0 ${PI}"/>
             <geometry>
                 <mesh filename="package://scara_description/meshes/ARM_HUB.stl" scale="0.001 0.001 0.001"/>
@@ -140,5 +140,5 @@
         <!-- elbow arm -->
         <visual>
-            <origin xyz="0 0 -0.003" rpy="${PI/2} 0 -${PI/2}"/>
+            <origin xyz="0 0 -0.0215" rpy="${PI/2} 0 -${PI/2}"/>
             <geometry>
                 <mesh filename="package://scara_description/meshes/MY_FOREARM.stl" scale="0.001 0.001 0.001"/>
@@ -147,5 +147,5 @@
         <!-- camera base-->
         <visual>
-            <origin xyz="0.1625 0.0195 0.011" rpy="${PI/2} 0 ${PI/2}"/>
+            <origin xyz="0.1625 0.0195 -0.0075" rpy="${PI/2} 0 ${PI/2}"/>
             <geometry>
                 <mesh filename="package://scara_description/meshes/MY_CAMERA_BASE.stl" scale="0.001 0.001 0.001"/>
@@ -154,5 +154,5 @@
         <!-- camera -->
         <visual>
-            <origin xyz="0.173 0.0195 0.011" rpy="${PI} 0 -${PI/2}"/>
+            <origin xyz="0.173 0.0195 -0.0075" rpy="${PI} 0 -${PI/2}"/>
             <geometry>
                 <mesh filename="package://scara_description/meshes/CAMERA.stl" scale="0.001 0.001 0.001"/>
@@ -160,5 +160,5 @@
         </visual>
         <collision>
-            <origin xyz="0 0 -0.003" rpy="${PI/2} 0 -${PI/2}"/>
+            <origin xyz="0 0 -0.0215" rpy="${PI/2} 0 -${PI/2}"/>
             <geometry>
                 <mesh filename="package://scara_description/meshes/MY_FOREARM.stl" scale="0.001 0.001 0.001"/>
@@ -167,5 +167,5 @@
         <xacro:default_inertial mass="1.5"/>
         <collision>
-            <origin xyz="0.1625 0.0195 0.011" rpy="${PI/2} 0 ${PI/2}"/>
+            <origin xyz="0.1625 0.0195 -0.0075" rpy="${PI/2} 0 ${PI/2}"/>
             <geometry>
                 <mesh filename="package://scara_description/meshes/MY_CAMERA_BASE.stl" scale="0.001 0.001 0.001"/>
@@ -176,5 +176,5 @@
     <link name="gripper_base">
         <visual>
-            <origin xyz="0 0 -0.0305" rpy="${PI/2} 0 0"/>
+            <origin xyz="0 0 -0.0430" rpy="${PI/2} 0 0"/>
             <geometry>
                 <mesh filename="package://scara_description/meshes/MY_GRIPPER_GEAR.stl" scale="0.001 0.001 0.001"/>
@@ -182,5 +182,5 @@
         </visual>
         <collision>
-            <origin xyz="0 0 -0.0305" rpy="${PI/2} 0 0"/>
+            <origin xyz="0 0 -0.0430" rpy="${PI/2} 0 0"/>
             <geometry>
                 <mesh filename="package://scara_description/meshes/MY_GRIPPER_GEAR.stl" scale="0.001 0.001 0.001"/>
@@ -191,5 +191,5 @@
     <link name="gripper">
         <visual>
-            <origin xyz="0 0 -0.015" rpy="${PI} 0 ${PI}"/>
+            <origin xyz="0 0 -0.0275" rpy="${PI} 0 ${PI}"/>
             <geometry>
                 <cylinder radius="0.004" length="0.065"/>
@@ -197,5 +197,5 @@
         </visual>
         <visual>
-            <origin xyz="0.005 0 -0.040" rpy="${PI} 0 ${PI}"/>
+            <origin xyz="0.005 0 -0.0525" rpy="${PI} 0 ${PI}"/>
             <geometry>
                 <box size="0.01 0.001 0.01"/>
@@ -203,5 +203,5 @@
         </visual>
         <collision>
-            <origin xyz="0 0 -0.015" rpy="${PI} 0 ${PI}"/>
+            <origin xyz="0 0 -0.0275" rpy="${PI} 0 ${PI}"/>
             <geometry>
                 <cylinder radius="0.004" length="0.05"/>
@@ -227,23 +227,19 @@
         <parent link="z_base"/>
         <child link="shoulder"/>
-        <!--<origin xyz="0.067 0 -0.0125" rpy="0 0 1.98"/>-->
-        <origin xyz="0.067 0 -0.0125" rpy="0 0 0"/>
+        <origin xyz="0.067 0 0" rpy="0 0 0"/>
         <axis xyz="0 0 1"/>
         <limit effort="${effort}" velocity="${velocity}" lower="-1.98" upper="1.98"/>
-        <!--<limit effort="${effort}" velocity="${velocity}" lower="-3.96" upper="0.0"/>-->
     </joint>
     <joint name="joint_3" type="revolute">
         <parent link="shoulder"/>
         <child link="elbow"/>
-        <!--<origin xyz="0.092 0 -0.006" rpy="0 0 -2.27"/>-->
-        <origin xyz="0.092 0 -0.006" rpy="0 0 0"/>
+        <origin xyz="0.0925 0 0" rpy="0 0 0"/>
         <axis xyz="0 0 1"/>
         <limit effort="${effort}" velocity="${velocity}" lower="-2.27" upper="2.27"/>
-        <!--<limit effort="${effort}" velocity="${velocity}" lower="0.0" upper="4.54"/>-->
     </joint>
     <joint name="joint_4" type="revolute">
         <parent link="elbow"/>
         <child link="gripper_base"/>
-        <origin xyz="0.1 0 0" rpy="0 0 0"/>
+        <origin xyz="0.102525 0 0" rpy="0 0 0"/>
         <axis xyz="0 0 1"/>
         <limit effort="${effort}" velocity="${velocity}" lower="-${PI}" upper="${PI}"/>

Commit message: Changes due to making robot higher, so the camera can see the whole puzzzle element

File: src/scara_description/urdf/scara.urdf.xacro (robot description, xacro)
@@ -31,45 +31,45 @@
         <!-- Rod 1 -->
         <visual>
-            <origin xyz="0.067 0 0.13" rpy="0 0 0"/>
-            <geometry>
-                <cylinder radius="0.004" length="0.250"/>
+            <origin xyz="0.067 0 0.168" rpy="0 0 0"/>
+            <geometry>
+                <cylinder radius="0.004" length="0.320"/>
             </geometry>
         </visual>
         <!-- Rod 2 -->
         <visual>
-            <origin xyz="-0.008 0.048 0.13" rpy="0 0 0"/>
-            <geometry>
-                <cylinder radius="0.004" length="0.250"/>
-            </geometry>
-        </visual>
-        <collision>
-            <origin xyz="-0.008 -0.048 0.13" rpy="0 0 0"/>
-            <geometry>
-                <cylinder radius="0.004" length="0.250"/>
+            <origin xyz="-0.008 0.048 0.168" rpy="0 0 0"/>
+            <geometry>
+                <cylinder radius="0.004" length="0.320"/>
+            </geometry>
+        </visual>
+        <collision>
+            <origin xyz="-0.008 -0.048 0.168" rpy="0 0 0"/>
+            <geometry>
+                <cylinder radius="0.004" length="0.320"/>
             </geometry>
         </collision>
         <!-- Rod 3 -->
         <visual>
-            <origin xyz="-0.008 -0.048 0.13" rpy="0 0 0"/>
-            <geometry>
-                <cylinder radius="0.004" length="0.250"/>
-            </geometry>
-        </visual>
-        <collision>
-            <origin xyz="-0.008 -0.048 0.13" rpy="0 0 0"/>
-            <geometry>
-                <cylinder radius="0.004" length="0.250"/>
+            <origin xyz="-0.008 -0.048 0.168" rpy="0 0 0"/>
+            <geometry>
+                <cylinder radius="0.004" length="0.320"/>
+            </geometry>
+        </visual>
+        <collision>
+            <origin xyz="-0.008 -0.048 0.168" rpy="0 0 0"/>
+            <geometry>
+                <cylinder radius="0.004" length="0.320"/>
             </geometry>
         </collision>
         <!-- Threaded Rod -->
         <visual>
-            <origin xyz="0 0 0.13" rpy="0 0 0"/>
-            <geometry>
-                <cylinder radius="0.004" length="0.250"/>
+            <origin xyz="0 0 0.200" rpy="0 0 0"/>
+            <geometry>
+                <cylinder radius="0.004" length="0.280"/>
             </geometry>
         </visual>
         <!-- Base cover -->
         <visual>
-            <origin xyz="0.017 0 0.308" rpy="-${PI/2} 0 -${PI/2}"/>
+            <origin xyz="0.017 0 0.382" rpy="-${PI/2} 0 -${PI/2}"/>
             <geometry>
                 <mesh filename="package://scara_description/meshes/TOP_TRIANGLE.stl" scale="0.001 0.001 0.001"/>
@@ -219,7 +219,7 @@
         <parent link="base_link"/>
         <child link="z_base"/>
-        <origin xyz="0 0 0.239" rpy="0 0 0"/>
-        <axis xyz="0 0 1"/>
-        <limit effort="1000" velocity="10" lower="-0.143" upper="0.0"/>
+        <origin xyz="0 0 0.310" rpy="0 0 0"/>
+        <axis xyz="0 0 1"/>
+        <limit effort="1000" velocity="10" lower="-0.221" upper="0.0"/>
         <dynamics damping="0.5" friction="0.5"/>
     </joint>
