Commit message: Adjustmets for placing puzzles in 2D

File: src/scara_description/urdf/scara.urdf.xacro (robot description, xacro)
@@ -154,61 +154,61 @@
             </geometry>
         </visual>
+        <collision>
+            <origin xyz="0 0 -0.0215" rpy="${PI/2} 0 -${PI/2}"/>
+            <geometry>
+                <mesh filename="package://scara_description/meshes/MY_FOREARM.stl" scale="0.001 0.001 0.001"/>
+            </geometry>
+        </collision>
+        <xacro:default_inertial mass="1.5"/>
+        <collision>
+            <origin xyz="0.1625 0.0195 -0.0075" rpy="${PI/2} 0 ${PI/2}"/>
+            <geometry>
+                <mesh filename="package://scara_description/meshes/MY_CAMERA_BASE.stl" scale="0.001 0.001 0.001"/>
+            </geometry>
+        </collision>
+        <xacro:default_inertial mass="1.5"/>
+    </link>
+    <link name="gripper_base">
+        <visual>
+            <origin xyz="0 0 -0.0430" rpy="${PI/2} 0 0"/>
+            <geometry>
+                <mesh filename="package://scara_description/meshes/MY_GRIPPER_GEAR.stl" scale="0.001 0.001 0.001"/>
+            </geometry>
+        </visual>
+        <collision>
+            <origin xyz="0 0 -0.0430" rpy="${PI/2} 0 0"/>
+            <geometry>
+                <mesh filename="package://scara_description/meshes/MY_GRIPPER_GEAR.stl" scale="0.001 0.001 0.001"/>
+            </geometry>
+        </collision>
+        <xacro:default_inertial mass="1.5"/>
+        <visual>
+            <origin xyz="0 0 -0.0275" rpy="${PI} 0 ${PI}"/>
+            <geometry>
+                <cylinder radius="0.004" length="0.065"/>
+            </geometry>
+        </visual>
+        <visual>
+            <origin xyz="0.005 0 -0.0525" rpy="${PI} 0 ${PI}"/>
+            <geometry>
+                <box size="0.01 0.001 0.01"/>
+            </geometry>
+        </visual>
+        <collision>
+            <origin xyz="0 0 -0.0275" rpy="${PI} 0 ${PI}"/>
+            <geometry>
+                <cylinder radius="0.004" length="0.05"/>
+            </geometry>
+        </collision>
+        <xacro:default_inertial mass="1.5"/>
+    </link>
+    <link name="camera">
         <!-- camera -->
         <visual>
-            <origin xyz="0.173 0.0195 -0.0075" rpy="${PI} 0 -${PI/2}"/>
+            <origin xyz="0.03 0.0195 -0.0075" rpy="${PI} 0 -${PI/2}"/>
             <geometry>
                 <mesh filename="package://scara_description/meshes/CAMERA.stl" scale="0.001 0.001 0.001"/>
             </geometry>
         </visual>
-        <collision>
-            <origin xyz="0 0 -0.0215" rpy="${PI/2} 0 -${PI/2}"/>
-            <geometry>
-                <mesh filename="package://scara_description/meshes/MY_FOREARM.stl" scale="0.001 0.001 0.001"/>
-            </geometry>
-        </collision>
-        <xacro:default_inertial mass="1.5"/>
-        <collision>
-            <origin xyz="0.1625 0.0195 -0.0075" rpy="${PI/2} 0 ${PI/2}"/>
-            <geometry>
-                <mesh filename="package://scara_description/meshes/MY_CAMERA_BASE.stl" scale="0.001 0.001 0.001"/>
-            </geometry>
-        </collision>
-        <xacro:default_inertial mass="1.5"/>
-    </link>
-    <link name="gripper_base">
-        <visual>
-            <origin xyz="0 0 -0.0430" rpy="${PI/2} 0 0"/>
-            <geometry>
-                <mesh filename="package://scara_description/meshes/MY_GRIPPER_GEAR.stl" scale="0.001 0.001 0.001"/>
-            </geometry>
-        </visual>
-        <collision>
-            <origin xyz="0 0 -0.0430" rpy="${PI/2} 0 0"/>
-            <geometry>
-                <mesh filename="package://scara_description/meshes/MY_GRIPPER_GEAR.stl" scale="0.001 0.001 0.001"/>
-            </geometry>
-        </collision>
-        <xacro:default_inertial mass="1.5"/>
-    </link>
-    <link name="gripper">
-        <visual>
-            <origin xyz="0 0 -0.0275" rpy="${PI} 0 ${PI}"/>
-            <geometry>
-                <cylinder radius="0.004" length="0.065"/>
-            </geometry>
-        </visual>
-        <visual>
-            <origin xyz="0.005 0 -0.0525" rpy="${PI} 0 ${PI}"/>
-            <geometry>
-                <box size="0.01 0.001 0.01"/>
-            </geometry>
-        </visual>
-        <collision>
-            <origin xyz="0 0 -0.0275" rpy="${PI} 0 ${PI}"/>
-            <geometry>
-                <cylinder radius="0.004" length="0.05"/>
-            </geometry>
-        </collision>
-        <xacro:default_inertial mass="1.5"/>
     </link>
     <!-- joints -->
@@ -248,7 +248,9 @@
     </joint>
     <joint name="joint_5" type="fixed">
-        <parent link="gripper_base"/>
-        <child link="gripper"/>
-        <origin xyz="0 0 0" rpy="0 0 0"/>
+        <parent link="elbow"/>
+        <child link="camera"/>
+        <origin xyz="0.142525 0 0" rpy="0 0 0"/>
+        <axis xyz="0 0 1"/>
+        <limit effort="${effort}" velocity="${velocity}" lower="-${PI}" upper="${PI}"/>
     </joint>
 </robot>

File: src/scara_description/urdf/scara_ros2_control.xacro (robot description, xacro)
@@ -10,5 +10,5 @@
       <hardware>
         <plugin>scara_controller/ScaraInterface</plugin>
-        <param name ="port">/dev/ttyACM0</param>
+        <param name ="port">/dev/ttyUSB0</param>
       </hardware>
     </xacro:unless>

Commit message: Added possibility to control suction cup

File: src/scara_description/urdf/scara.urdf.xacro (robot description, xacro)
@@ -190,5 +190,5 @@
         </visual>
         <visual>
-            <origin xyz="0.005 0 -0.0525" rpy="${PI} 0 ${PI}"/>
+            <origin xyz="0.0035 0 -0.0525" rpy="${PI} 0 ${PI}"/>
             <geometry>
                 <box size="0.01 0.001 0.01"/>
@@ -204,9 +204,16 @@
     </link>
     <link name="camera">
-        <!-- camera -->
         <visual>
             <origin xyz="0.03 0.0195 -0.0075" rpy="${PI} 0 -${PI/2}"/>
             <geometry>
                 <mesh filename="package://scara_description/meshes/CAMERA.stl" scale="0.001 0.001 0.001"/>
+            </geometry>
+        </visual>
+    </link>
+    <link name="suction_cup">
+        <visual>
+            <origin xyz="0 0 -0.06" rpy="${PI} 0 ${PI}"/>
+            <geometry>
+                <cylinder radius="0.008" length="0.005"/>
             </geometry>
         </visual>
@@ -247,4 +254,5 @@
         <limit effort="${effort}" velocity="${velocity}" lower="-${PI}" upper="${PI}"/>
     </joint>
+    <!-- joint_5 is a fake joint to allow camera positioning-->
     <joint name="joint_5" type="fixed">
         <parent link="elbow"/>
@@ -254,3 +262,11 @@
         <limit effort="${effort}" velocity="${velocity}" lower="-${PI}" upper="${PI}"/>
     </joint>
+    <!-- joint_6 is a fake ravolute joint to allow scara_interface to controll suction gripper state-->
+    <joint name="joint_6" type="revolute">
+        <parent link="gripper_base"/>
+        <child link="suction_cup"/>
+        <origin xyz="0 0 0" rpy="0 0 0"/>
+        <axis xyz="0 0 1"/>
+        <limit effort="${effort}" velocity="${velocity}" lower="0.0" upper="${PI}"/>
+    </joint>
 </robot>

File: src/scara_description/urdf/scara_ros2_control.xacro (robot description, xacro)
@@ -29,4 +29,8 @@
       <state_interface name="position"/>
     </joint>
+    <joint name="joint_6">
+      <command_interface name="position"/>
+      <state_interface name="position"/>
+    </joint>
   </ros2_control>
 </robot>

Commit message: Testing assembly procedure.

File: src/scara_description/urdf/scara.urdf.xacro (robot description, xacro)
@@ -230,5 +230,5 @@
         <origin xyz="0 0 0.310" rpy="0 0 0"/>
         <axis xyz="0 0 1"/>
-        <limit effort="1000" velocity="10" lower="-0.221" upper="0.0"/>
+        <limit effort="1000" velocity="10" lower="-0.221" upper="0.001"/>
         <dynamics damping="0.5" friction="0.5"/>
     </joint>

Commit message: Adjustments, trying to fix pickup-position error

File: src/scara_description/urdf/scara.urdf.xacro (robot description, xacro)
@@ -238,5 +238,5 @@
         <origin xyz="0.067 0 0" rpy="0 0 0"/>
         <axis xyz="0 0 1"/>
-        <limit effort="${effort}" velocity="${velocity}" lower="-1.98" upper="1.98"/>
+        <limit effort="${effort}" velocity="${velocity}" lower="-1.9635" upper="1.9635"/>
     </joint>
     <joint name="joint_3" type="revolute">

Commit message: Simplified STL model naming. Created better readme.

File: src/scara_description/urdf/scara.urdf.xacro (robot description, xacro)
@@ -107,5 +107,5 @@
             <origin xyz="0 0 -0.0125" rpy="0 0 0"/>
             <geometry>
-                <mesh filename="package://scara_description/meshes/MY_ARM_TOP.stl" scale="0.001 0.001 0.001"/>
+                <mesh filename="package://scara_description/meshes/ARM_TOP.stl" scale="0.001 0.001 0.001"/>
             </geometry>
         </visual>
@@ -113,5 +113,5 @@
             <origin xyz="0 0 -0.0125" rpy="0 0 0"/>
             <geometry>
-                <mesh filename="package://scara_description/meshes/MY_ARM_TOP.stl" scale="0.001 0.001 0.001"/>
+                <mesh filename="package://scara_description/meshes/ARM_TOP.stl" scale="0.001 0.001 0.001"/>
             </geometry>
         </collision>
@@ -120,5 +120,5 @@
             <origin xyz="0 0 -0.0415" rpy="${PI/2} 0 -${PI/2} "/>
             <geometry>
-                <mesh filename="package://scara_description/meshes/MY_ARM_BOTTOM.stl" scale="0.001 0.001 0.001"/>
+                <mesh filename="package://scara_description/meshes/ARM_BOTTOM.stl" scale="0.001 0.001 0.001"/>
             </geometry>
         </visual>
@@ -144,5 +144,5 @@
             <origin xyz="0 0 -0.0215" rpy="${PI/2} 0 -${PI/2}"/>
             <geometry>
-                <mesh filename="package://scara_description/meshes/MY_FOREARM.stl" scale="0.001 0.001 0.001"/>
+                <mesh filename="package://scara_description/meshes/FOREARM.stl" scale="0.001 0.001 0.001"/>
             </geometry>
         </visual>
@@ -151,5 +151,5 @@
             <origin xyz="0.1625 0.0195 -0.0075" rpy="${PI/2} 0 ${PI/2}"/>
             <geometry>
-                <mesh filename="package://scara_description/meshes/MY_CAMERA_BASE.stl" scale="0.001 0.001 0.001"/>
+                <mesh filename="package://scara_description/meshes/CAMERA_BASE.stl" scale="0.001 0.001 0.001"/>
             </geometry>
         </visual>
@@ -157,5 +157,5 @@
             <origin xyz="0 0 -0.0215" rpy="${PI/2} 0 -${PI/2}"/>
             <geometry>
-                <mesh filename="package://scara_description/meshes/MY_FOREARM.stl" scale="0.001 0.001 0.001"/>
+                <mesh filename="package://scara_description/meshes/FOREARM.stl" scale="0.001 0.001 0.001"/>
             </geometry>
         </collision>
@@ -164,5 +164,5 @@
             <origin xyz="0.1625 0.0195 -0.0075" rpy="${PI/2} 0 ${PI/2}"/>
             <geometry>
-                <mesh filename="package://scara_description/meshes/MY_CAMERA_BASE.stl" scale="0.001 0.001 0.001"/>
+                <mesh filename="package://scara_description/meshes/CAMERA_BASE.stl" scale="0.001 0.001 0.001"/>
             </geometry>
         </collision>
@@ -173,5 +173,5 @@
             <origin xyz="0 0 -0.0430" rpy="${PI/2} 0 0"/>
             <geometry>
-                <mesh filename="package://scara_description/meshes/MY_GRIPPER_GEAR.stl" scale="0.001 0.001 0.001"/>
+                <mesh filename="package://scara_description/meshes/GRIPPER_GEAR.stl" scale="0.001 0.001 0.001"/>
             </geometry>
         </visual>
@@ -179,5 +179,5 @@
             <origin xyz="0 0 -0.0430" rpy="${PI/2} 0 0"/>
             <geometry>
-                <mesh filename="package://scara_description/meshes/MY_GRIPPER_GEAR.stl" scale="0.001 0.001 0.001"/>
+                <mesh filename="package://scara_description/meshes/GRIPPER_GEAR.stl" scale="0.001 0.001 0.001"/>
             </geometry>
         </collision>
